File: KNOB_PANEL.kicad_pcb (KiCad board)
At the start: 2 copper layers, 100 x 50 mm, 6 parts

Commit message: Add specific custom number on panel
Other:
- board text added: "JLCJLCJLCJLC"
Changed lines of the file:
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@@
   (general
     (thickness 1.6)
-    (drawings 32)
+    (drawings 33)
     (tracks 0)
     (zones 0)
@@
     (pad 1 np_thru_hole circle (at 0 0) (size 3.2 3.2) (drill 3.2) (layers *.Cu *.Mask))
   )
+  (gr_text JLCJLCJLCJLC (at 192 96.25) (layer B.SilkS)
+    (effects (font (size 1 1) (thickness 0.15)) (justify left mirror))
+  )
   (gr_text "KNOB_PANEL V1.0 by XiNGRZ" (at 192 98) (layer B.SilkS)
